File: MiniSirius.kicad_sch (KiCad schematic)
At the start: 67 parts, among them J1 Conn_Coaxial_SMA, J2 JST_03, J4 JST_04, J5 Molex_MCRF_73412-0110, J6 JST_03, J7 JST_02, J8 JST_02, Q1 BSS138, SW3 Slide_Switch_SPDT, U1 RFM95W-868S2, U2 MAX-M10S, U4 L7805, U5 DRV8870DDA

Commit message: update schematic
Parts:
- removed C5: NC, Capacitor_SMD:C_0603_1608Metric_Pad1.08x0.95mm_HandSolder, symbol Device:C
- removed J4: JST_04, Connector_JST:JST_EH_S4B-EH_1x04_P2.50mm_Horizontal, symbol PCM_SL_Connectors:JST_04
- removed J5: Molex_MCRF_73412-0110, Connector_Coaxial:U.FL_Molex_MCRF_73412-0110_Vertical, symbol Connector:Conn_Coaxial
- removed J8: JST_02, Connector_JST:JST_EH_B2B-EH-A_1x02_P2.50mm_Vertical, symbol PCM_SL_Connectors:JST_02
- removed L2, L3: NC, Inductor_SMD:L_0603_1608Metric_Pad1.05x0.95mm_HandSolder, symbol Device:L
- removed R29, R30: 0R, Resistor_SMD:R_0603_1608Metric_Pad0.98x0.95mm_HandSolder, symbol Device:R
- removed U2: MAX-M10S, RF_GPS:ublox_MAX, symbol RF_GPS:MAX-M10S
- added J10, J11, J4, J9: JST_03, Connector_JST:JST_EH_B3B-EH-A_1x03_P2.50mm_Vertical, symbol PCM_SL_Connectors:JST_03
- added J20, J8: JST_04, Connector_JST:JST_EH_S4B-EH_1x04_P2.50mm_Horizontal, symbol PCM_SL_Connectors:JST_04
- added J5: JST_02, Connector_JST:JST_EH_B2B-EH-A_1x02_P2.50mm_Vertical, symbol PCM_SL_Connectors:JST_02
- added R75, R76: 0R, Resistor_SMD:R_0603_1608Metric_Pad0.98x0.95mm_HandSolder, symbol Device:R
- added U2: DRV8870DDA, Package_SO:Texas_HTSOP-8-1EP_3.9x4.9mm_P1.27mm_EP2.95x4.9mm_Mask2.4x3.1mm_ThermalVias, symbol Driver_Motor:DRV8870DDA
- added U9: SAM-M1_10Q-00B, SAM-M10Q-00B:XCVR_SAM-M10Q-00B, symbol SAM-M10Q-00B:SAM-M10Q-00B
- C3, C4: value NC -> 0.1µF
- R26: value NC -> 0.2R
Connections:
- net +3V3: now also J10.2, J11.2, J20.3, J4.2, J8.3, J9.2, R75.1, R76.1, U2.4 (VREF); no longer R17.1, R18.1
- net GND: now also R26.2, J10.3, J11.3, J20.4, J4.3, J8.4, J9.3, U2.1 (GND), U2.9 (GND), U9.1 (GND), U9.10 (GND), U9.11 (GND), U9.15 (GND), U9.16 (GND), U9.20 (GND), U9.4 (GND), U9.5 (GND), U9.6 (GND); no longer J7.2
- net PPS: now also R17.2
- net PWM_1: now also J9.1; no longer J2.1
- net RX_GPS: now also R15.2; no longer R12.1
- net SCL0: now also R13.2, J8.2; no longer R15.1
- net SCL1: now also J20.2
- net SDA0: now also R12.2, J8.1; no longer R14.1
- net SDA1: now also J20.1
- net TX_GPS: now also R14.2; no longer R13.1
- net VBAT: now also C3.1, C4.1, U2.5 (VM)
- net V_BCKP: now also R18.2
- net at U5.8 (OUT2): now also J7.2
- net M2_2: now reaches A1.24 (GP18)
- net M2_2: now also U2.2 (IN2)
- net M1_1: now reaches A1.29 (GP22)
- net M1_1: now also U5.3 (IN1)
- net GP28: now reaches A1.34 (ADC2/GP28)
- net GP28: now also J10.1
- net GP2: now reaches A1.4 (GP2)
- net GP2: now also J11.1
- net at R11.2: now also U9.18 (~{RESET})
- net at R10.2: now also U9.8 (~{SAFEBOOT})
- net at R9.2: now also U9.19 (EXTINT)
- net M1 renamed M1_2
- net M1_2: now also U5.2 (IN2); no longer U5.3 (IN1)
- net M2 renamed M2_1
- net M2_1: now also U2.3 (IN1); no longer U5.2 (IN2)
- net VCC_RF: no longer names the net of R26.1
- net VCC_RF: now also U2.7 (ISEN)
- new net: R75.2, U9.17 (VCC)
- new net: R13.1, U9.12 (SCL)
- new net: R14.1, U9.13 (TXD)
- new net: R15.1, U9.14 (RXD)
- new net: R76.2, U9.2 (V_IO)
- new net: R18.1, U9.3 (V_BCKP)
- new net: R17.1, U9.7 (TIMEPULSE)
- new net: R12.1, U9.9 (SDA)
- new net: J5.1, U2.6 (OUT1)
- new net: J5.2, U2.8 (OUT2)
- new net GP18: J2.1
- new net GP22: J4.1
- no-connect marks 13 -> 10
Other:
- note removed: "GPS Antenna"
- moved on the sheet: C8, C9, J7, R31, U5
