File: Sensors.kicad_sch (KiCad schematic)
At the start: 7 parts, among them U3 SX1509BIULTRT, U6 LSM6DSL

Commit message: update schematic
Parts:
- added R55, R56, R57, R58, R59, R60, R61, R62, R63, R64, R65, R66, R67, R68, R69, R70, R71, R72, R73: 0R, Resistor_SMD:R_0603_1608Metric_Pad0.98x0.95mm_HandSolder, symbol Device:R
Connections:
- net +3V3: now also R55.1, R59.2, R60.2, R70.2, R71.2; no longer A2.1 (VDD_IO), A2.10 (VDD), A2.6 (CS), U6.5 (VDDIO), U6.8 (VDD)
- net GND: now also R58.1, R62.2, R63.1, R64.1, R65.1; no longer A2.3 (RESERVED), A2.5 (SDO/SA0), U6.1 (SDO/SA0), U6.2 (SDX), U6.3 (SCX)
- net INT1_IMU: now also R68.2; no longer U6.4 (INT1)
- net INT2_IMU: now also R69.2; no longer U6.9 (INT2)
- net INT_BARO: now also R61.2; no longer A2.7 (INT_DRDY)
- net SCL0: now also R56.1, R67.1, R73.1; no longer A2.2 (SCL/SPC), U3.25 (SCL), U6.13 (SCL)
- net SDA0: now also R57.1, R66.1, R72.1; no longer A2.4 (SDA/SDI/SDO), U3.24 (SDA), U6.14 (SDA)
- new net: R70.1, U6.8 (VDD)
- new net: R64.2, U6.2 (SDX)
- new net: A2.5 (SDO/SA0), R58.2
- new net: R66.2, U6.14 (SDA)
- new net: A2.10 (VDD), R60.1
- new net: A2.2 (SCL/SPC), R56.2
- new net: R67.2, U6.13 (SCL)
- new net: A2.3 (RESERVED), R62.1
- new net: R65.2, U6.3 (SCX)
- new net: R72.2, U3.24 (SDA)
- new net: R73.2, U3.25 (SCL)
- new net: R63.2, U6.1 (SDO/SA0)
- new net: A2.6 (CS), R55.2
- new net: R68.1, U6.4 (INT1)
- new net: R71.1, U6.5 (VDDIO)
- new net: R69.1, U6.9 (INT2)
- new net: A2.1 (VDD_IO), R59.1
- new net: A2.4 (SDA/SDI/SDO), R57.2
- new net: A2.7 (INT_DRDY), R61.1
- no-connect marks 0 -> 17
