File: interuption.kicad_sch (KiCad schematic)
At the start: 32 parts, among them J12 JST_02, J13 JST_02, J3 JST_02, SW1 Push_Button, SW2 Push_Button, U7 SX1509BIULTRT, U8 74HC14

Commit message: update schematic
Parts:
- added J14, J15, J16, J17, J18, J19: JST_03, Connector_JST:JST_EH_B3B-EH-A_1x03_P2.50mm_Vertical, symbol PCM_SL_Connectors:JST_03
- added SW4: SW_Push_SPDT, symbol Switch:SW_Push_SPDT
Connections:
- net +3V3: now also J3.2, SW1.1, SW2.1, J14.2, J15.2, J16.2, J17.2, J18.2, J19.2, SW4.2 (B); no longer R19.2, R2.2, R53.1
- net GND: now also R19.1, R2.1, R53.2, J14.3, J15.3, J16.3, J17.3, J18.3, J19.3, SW4.3 (C); no longer J3.1, SW1.2, SW2.2
- net IO1_3: no longer U7.6 (I/O[5])
- net IO1_5: now also U7.6 (I/O[5])
- net RBF: now also J3.1, R53.1; no longer J3.2, R53.2
- net Rotation_Switch: now reaches C16.1, R48.1, U8.11
- net Rotation_Switch: now also SW4.1 (A)
- net SHM5: now reaches C17.1, R49.1, U8.13
- net SHM5: now also J19.1
- net IO1_8: now reaches U7.13 (I/O[8])
- net IO1_8: now also J18.1
- net IO1_9: now reaches U7.14 (I/O[9])
- net IO1_9: now also J17.1
- net IO1_10: now reaches U7.15 (I/O[10])
- net IO1_10: now also J16.1
- net IO1_11: now reaches U7.16 (I/O[11])
- net IO1_11: now also J15.1
- net M1_Button renamed M1_1_Button
- net M1_1_Button: now also R2.2, SW1.2; no longer R2.1, SW1.1
- net M2_Button renamed M2_1_Button
- net M2_1_Button: now also R19.2, SW2.2; no longer R19.1, SW2.1
- new net IO1_12: J14.1
- no-connect marks 0 -> 7
Other:
- note added: "RBF & Jack"
- note added: "Rotation Selector"
- note removed: "RBF & Jack Pull-Up"
- moved on the sheet: J3, R2, R39, R40, R53, SW1, U7
